Commit message: initial commit

File: eklavya5_description/robots/chasisss.URDF (robot description, URDF)
Before this commit: robot chasisss, 6 links, 5 joints
Links:
- added link camera_link, mass 1e-5; collision box size=0.05 0.05 0.05; visual box size=0.05 0.05 0.05
Joints:
- added joint camera_joint: type fixed, parent Steering, child camera_link, origin xyz=0.05 0 0.5 rpy=0 0 0, axis 0 1 0

File: eklavya5_description/robots/chasisss_sample.urdf (robot description, URDF)
Before this commit: robot eklavya, 8 links, 7 joints
Links:
- link back_left_wheel: geometry collision cylinder length=0.1143 radius=0.17775; visual mesh filename=package://eklavya5_description/meshes/wheel.stl
- link back_right_wheel: geometry collision cylinder length=0.1143 radius=0.17775; visual mesh filename=package://eklavya5_description/meshes/wheel.stl
- link base_link: geometry collision box size=1.0074 0.5709 0.2675; visual mesh filename=package://eklavya5_description/meshes/base_link.stl
- link base_link_user_rail_part: geometry collision box size=0.001 0.001 0.001; visual mesh filename=package://eklavya5_description/meshes/user_rail.stl
- link front_left_wheel: geometry collision cylinder length=0.1143 radius=0.17775; visual mesh filename=package://eklavya5_description/meshes/wheel.stl
- link front_right_wheel: geometry collision cylinder length=0.1143 radius=0.17775; visual mesh filename=package://eklavya5_description/meshes/wheel.stl
